File: USB-Audio_ver_1_0.brd (EAGLE design)
At the start: 49 x 30 mm, 61 parts, among them IC1 PCM2904DB, IC2 OPA2353UA, IC3 OPA2353UA, IC4 REG103GA-A

Commit message: Modified power supply and silk printing
Parts:
- moved C25 3.19 mm to (-15.9, -7.94)
- moved R5 1.62 mm to (-15.9, -10.2)
- moved C24 0.71 mm to (-15.9, -5.71)
Connections:
- net +5V: no longer R5.1
- net GND: now also R5.1
Routing:
- net +5V: track 58.2 -> 40.5 mm, vias 3 -> 2
- net VCOM: track 52.6 -> 41.7 mm, vias 2 -> 3
- net XTO: track 17.3 -> 26.2 mm, vias 2 -> 0
- net SSPND: track 53.9 -> 46.1 mm, vias 2 -> 3
- net N$14: track 48.2 -> 43.1 mm
- net VINL: track 11.4 -> 6.84 mm, vias 0 -> 1
- net N$4: track 10.9 -> 6.66 mm
- net V+: track 76.5 -> 75.4 mm
- net N$15: track 14.4 -> 13.4 mm
- net B_FUSE_USB_MINI_B: track 13.4 -> 12.8 mm
Other:
- board text added: "+"
- board text added: "-"
- board text added: "Input L"
- board text added: "Input R"
- board text added: "Output R"
- board text added: "USB-Audio Ver. 1.0 Designed by Masato Kubotera on November 23, 2022."
- board text removed: "USB-Audio Ver. 1.0 Designed by Masato Kubotera on November 15, 2022."
